File: dummy-load.sch (EAGLE design)
At the start: 71 parts, among them T1 BU931P, T2 BU931P, T3 BU931P, T4 BU931P, T5 BU931P, T6 BU931P, T7 BU931P, T8 BU931P, U1 TLV272CD, U10 MCP4725A0T-E/CH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

Commit message: PCB routing
Connections:
- net A1: now also X1-1.KL; no longer X1-9.KL
- net A2: now also X1-2.KL; no longer X1-10.KL
- net A3: now also X1-3.KL; no longer X1-11.KL
- net A4: now also X1-4.KL; no longer X1-12.KL
- net A5: now also X1-16.KL; no longer X1-13.KL
- net A6: now also X1-15.KL; no longer X1-14.KL
- net A7: now also X1-14.KL; no longer X1-15.KL
- net A8: now also X1-13.KL; no longer X1-16.KL
- net I1: now also X1-5.KL; no longer X1-1.KL
- net I2: now also X1-6.KL; no longer X1-2.KL
- net I3: now also X1-7.KL; no longer X1-3.KL
- net I4: now also X1-8.KL; no longer X1-4.KL
- net I5: now also X1-12.KL; no longer X1-5.KL
- net I6: now also X1-11.KL; no longer X1-6.KL
- net I7: now also X1-10.KL; no longer X1-7.KL
- net I8: now also X1-9.KL; no longer X1-8.KL
Other:
- moved on the sheet: H1, H2, H3, H4
Changed lines of the file:
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@@
 <attribute name="VALUE" x="43.18" y="-50.8" size="1.778" layer="96" rot="R180"/>
 </instance>
-<instance part="H1" gate="G$1" x="33.02" y="-17.78" smashed="yes">
-<attribute name="NAME" x="35.052" y="-17.1958" size="1.778" layer="95"/>
-<attribute name="VALUE" x="35.052" y="-20.2438" size="1.778" layer="96"/>
+<instance part="H1" gate="G$1" x="40.64" y="-17.78" smashed="yes">
+<attribute name="NAME" x="42.672" y="-17.1958" size="1.778" layer="95"/>
+<attribute name="VALUE" x="42.672" y="-20.2438" size="1.778" layer="96"/>
 </instance>
-<instance part="H2" gate="G$1" x="33.02" y="-25.4" smashed="yes">
-<attribute name="NAME" x="35.052" y="-24.8158" size="1.778" layer="95"/>
-<attribute name="VALUE" x="35.052" y="-27.8638" size="1.778" layer="96"/>
+<instance part="H2" gate="G$1" x="40.64" y="-25.4" smashed="yes">
+<attribute name="NAME" x="42.672" y="-24.8158" size="1.778" layer="95"/>
+<attribute name="VALUE" x="42.672" y="-27.8638" size="1.778" layer="96"/>
 </instance>
-<instance part="H3" gate="G$1" x="33.02" y="-33.02" smashed="yes">
-<attribute name="NAME" x="35.052" y="-32.4358" size="1.778" layer="95"/>
-<attribute name="VALUE" x="35.052" y="-35.4838" size="1.778" layer="96"/>
+<instance part="H3" gate="G$1" x="40.64" y="-33.02" smashed="yes">
+<attribute name="NAME" x="42.672" y="-32.4358" size="1.778" layer="95"/>
+<attribute name="VALUE" x="42.672" y="-35.4838" size="1.778" layer="96"/>
 </instance>
-<instance part="H4" gate="G$1" x="33.02" y="-40.64" smashed="yes">
-<attribute name="NAME" x="35.052" y="-40.0558" size="1.778" layer="95"/>
-<attribute name="VALUE" x="35.052" y="-43.1038" size="1.778" layer="96"/>
+<instance part="H4" gate="G$1" x="40.64" y="-40.64" smashed="yes">
+<attribute name="NAME" x="42.672" y="-40.0558" size="1.778" layer="95"/>
+<attribute name="VALUE" x="42.672" y="-43.1038" size="1.778" layer="96"/>
 </instance>
 </instances>
@@
 </segment>
 <segment>
-<pinref part="X1" gate="-5" pin="KL"/>
-<wire x1="22.86" y1="-27.94" x2="15.24" y2="-27.94" width="0.1524" layer="91"/>
-<label x="20.32" y="-27.94" size="1.778" layer="95"/>
+<pinref part="X1" gate="-12" pin="KL"/>
+<wire x1="20.32" y1="-45.72" x2="15.24" y2="-45.72" width="0.1524" layer="91"/>
+<label x="17.78" y="-45.72" size="1.778" layer="95"/>
 </segment>
 </net>
@@
 </segment>
 <segment>
-<pinref part="X1" gate="-9" pin="KL"/>
-<wire x1="22.86" y1="-38.1" x2="15.24" y2="-38.1" width="0.1524" layer="91"/>
-<label x="20.32" y="-38.1" size="1.778" layer="95"/>
+<pinref part="X1" gate="-1" pin="KL"/>
+<wire x1="15.24" y1="-17.78" x2="20.32" y2="-17.78" width="0.1524" layer="91"/>
+<label x="17.78" y="-17.78" size="1.778" layer="95"/>
 </segment>
 </net>
@@
 </segment>
 <segment>
-<pinref part="X1" gate="-6" pin="KL"/>
-<wire x1="15.24" y1="-30.48" x2="22.86" y2="-30.48" width="0.1524" layer="91"/>
-<label x="20.32" y="-30.48" size="1.778" layer="95"/>
+<pinref part="X1" gate="-11" pin="KL"/>
+<wire x1="20.32" y1="-43.18" x2="15.24" y2="-43.18" width="0.1524" layer="91"/>
+<label x="17.78" y="-43.18" size="1.778" layer="95"/>
 </segment>
 </net>
@@
 </segment>
 <segment>
-<pinref part="X1" gate="-7" pin="KL"/>
-<wire x1="22.86" y1="-33.02" x2="15.24" y2="-33.02" width="0.1524" layer="91"/>
-<label x="20.32" y="-33.02" size="1.778" layer="95"/>
+<pinref part="X1" gate="-10" pin="KL"/>
+<wire x1="20.32" y1="-40.64" x2="15.24" y2="-40.64" width="0.1524" layer="91"/>
+<label x="17.78" y="-40.64" size="1.778" layer="95"/>
 </segment>
 </net>
@@
 </segment>
 <segment>
-<pinref part="X1" gate="-8" pin="KL"/>
-<wire x1="15.24" y1="-35.56" x2="22.86" y2="-35.56" width="0.1524" layer="91"/>
-<label x="20.32" y="-35.56" size="1.778" layer="95"/>
+<pinref part="X1" gate="-9" pin="KL"/>
+<wire x1="15.24" y1="-38.1" x2="20.32" y2="-38.1" width="0.1524" layer="91"/>
+<label x="17.78" y="-38.1" size="1.778" layer="95"/>
 </segment>
 </net>
@@
 </segment>
 <segment>
-<pinref part="X1" gate="-1" pin="KL"/>
-<wire x1="15.24" y1="-17.78" x2="22.86" y2="-17.78" width="0.1524" layer="91"/>
-<label x="20.32" y="-17.78" size="1.778" layer="95"/>
+<pinref part="X1" gate="-5" pin="KL"/>
+<wire x1="15.24" y1="-27.94" x2="20.32" y2="-27.94" width="0.1524" layer="91"/>
+<label x="17.78" y="-27.94" size="1.778" layer="95"/>
 </segment>
 </net>
@@
 </segment>
 <segment>
-<pinref part="X1" gate="-2" pin="KL"/>
-<wire x1="15.24" y1="-20.32" x2="22.86" y2="-20.32" width="0.1524" layer="91"/>
-<label x="20.32" y="-20.32" size="1.778" layer="95"/>
+<pinref part="X1" gate="-6" pin="KL"/>
+<wire x1="20.32" y1="-30.48" x2="15.24" y2="-30.48" width="0.1524" layer="91"/>
+<label x="17.78" y="-30.48" size="1.778" layer="95"/>
 </segment>
 </net>
@@
 </segment>
 <segment>
-<pinref part="X1" gate="-3" pin="KL"/>
-<wire x1="22.86" y1="-22.86" x2="15.24" y2="-22.86" width="0.1524" layer="91"/>
-<label x="20.32" y="-22.86" size="1.778" layer="95"/>
+<pinref part="X1" gate="-7" pin="KL"/>
+<wire x1="15.24" y1="-33.02" x2="20.32" y2="-33.02" width="0.1524" layer="91"/>
+<label x="17.78" y="-33.02" size="1.778" layer="95"/>
 </segment>
 </net>
@@
 </segment>
 <segment>
-<pinref part="X1" gate="-4" pin="KL"/>
-<wire x1="15.24" y1="-25.4" x2="22.86" y2="-25.4" width="0.1524" layer="91"/>
-<label x="20.32" y="-25.4" size="1.778" layer="95"/>
+<pinref part="X1" gate="-8" pin="KL"/>
+<wire x1="20.32" y1="-35.56" x2="15.24" y2="-35.56" width="0.1524" layer="91"/>
+<label x="17.78" y="-35.56" size="1.778" layer="95"/>
 </segment>
 </net>
@@
 </segment>
 <segment>
-<pinref part="X1" gate="-10" pin="KL"/>
-<wire x1="15.24" y1="-40.64" x2="22.86" y2="-40.64" width="0.1524" layer="91"/>
-<label x="20.32" y="-40.64" size="1.778" layer="95"/>
+<pinref part="X1" gate="-2" pin="KL"/>
+<wire x1="15.24" y1="-20.32" x2="20.32" y2="-20.32" width="0.1524" layer="91"/>
+<label x="17.78" y="-20.32" size="1.778" layer="95"/>
 </segment>
 </net>
@@
 </segment>
 <segment>
-<pinref part="X1" gate="-11" pin="KL"/>
-<wire x1="22.86" y1="-43.18" x2="15.24" y2="-43.18" width="0.1524" layer="91"/>
-<label x="20.32" y="-43.18" size="1.778" layer="95"/>
+<pinref part="X1" gate="-3" pin="KL"/>
+<wire x1="15.24" y1="-22.86" x2="20.32" y2="-22.86" width="0.1524" layer="91"/>
+<label x="17.78" y="-22.86" size="1.778" layer="95"/>
 </segment>
 </net>
@@
 </segment>
 <segment>
-<pinref part="X1" gate="-12" pin="KL"/>
-<wire x1="15.24" y1="-45.72" x2="22.86" y2="-45.72" width="0.1524" layer="91"/>
-<label x="20.32" y="-45.72" size="1.778" layer="95"/>
+<pinref part="X1" gate="-4" pin="KL"/>
+<wire x1="20.32" y1="-25.4" x2="15.24" y2="-25.4" width="0.1524" layer="91"/>
+<label x="17.78" y="-25.4" size="1.778" layer="95"/>
 </segment>
 </net>
@@
 </segment>
 <segment>
-<pinref part="X1" gate="-13" pin="KL"/>
-<wire x1="22.86" y1="-48.26" x2="15.24" y2="-48.26" width="0.1524" layer="91"/>
-<label x="20.32" y="-48.26" size="1.778" layer="95"/>
+<pinref part="X1" gate="-16" pin="KL"/>
+<wire x1="20.32" y1="-55.88" x2="15.24" y2="-55.88" width="0.1524" layer="91"/>
+<label x="17.78" y="-55.88" size="1.778" layer="95"/>
 </segment>
 </net>
@@
 </segment>
 <segment>
-<pinref part="X1" gate="-14" pin="KL"/>
-<wire x1="15.24" y1="-50.8" x2="22.86" y2="-50.8" width="0.1524" layer="91"/>
-<label x="20.32" y="-50.8" size="1.778" layer="95"/>
+<pinref part="X1" gate="-15" pin="KL"/>
+<wire x1="20.32" y1="-53.34" x2="15.24" y2="-53.34" width="0.1524" layer="91"/>
+<label x="17.78" y="-53.34" size="1.778" layer="95"/>
 </segment>
 </net>
@@
 </segment>
 <segment>
-<pinref part="X1" gate="-15" pin="KL"/>
-<wire x1="22.86" y1="-53.34" x2="15.24" y2="-53.34" width="0.1524" layer="91"/>
-<label x="20.32" y="-53.34" size="1.778" layer="95"/>
+<pinref part="X1" gate="-14" pin="KL"/>
+<wire x1="20.32" y1="-50.8" x2="15.24" y2="-50.8" width="0.1524" layer="91"/>
+<label x="17.78" y="-50.8" size="1.778" layer="95"/>
 </segment>
 </net>
@@
 </segment>
 <segment>
-<pinref part="X1" gate="-16" pin="KL"/>
-<wire x1="15.24" y1="-55.88" x2="22.86" y2="-55.88" width="0.1524" layer="91"/>
-<label x="20.32" y="-55.88" size="1.778" layer="95"/>
-</segment>
-</net>
+<pinref part="X1" gate="-13" pin="KL"/>
+<wire x1="20.32" y1="-48.26" x2="15.24" y2="-48.26" width="0.1524" layer="91"/>
+<label x="17.78" y="-48.26" size="1.778" layer="95"/>
+</segment>
+</net>

Commit message: Add XT60 connector
Parts:
- added P1: XT60M-H, dummy-load:XT60M-H
Connections:
- net AGND: now also P1.2
- net VCC: now also P1.1
Other:
- moved on the sheet: H1, H2, H3, H4
Changed lines of the file:
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@@
 <part name="H3" library="holes" library_urn="urn:adsk.eagle:library:237" deviceset="MOUNT-HOLE" device="3.6" package3d_urn="urn:adsk.eagle:package:14272/1"/>
 <part name="H4" library="holes" library_urn="urn:adsk.eagle:library:237" deviceset="MOUNT-HOLE" device="3.6" package3d_urn="urn:adsk.eagle:package:14272/1"/>
+<part name="P1" library="dummy-load" deviceset="XT60M-H" device=""/>
+<part name="P+10" library="supply1" library_urn="urn:adsk.eagle:library:371" deviceset="VCC" device=""/>
+<part name="AGND30" library="supply1" library_urn="urn:adsk.eagle:library:371" deviceset="AGND" device=""/>
 </parts>
 <sheets>
@@
 <attribute name="VALUE" x="43.18" y="-50.8" size="1.778" layer="96" rot="R180"/>
 </instance>
-<instance part="H1" gate="G$1" x="40.64" y="-17.78" smashed="yes">
-<attribute name="NAME" x="42.672" y="-17.1958" size="1.778" layer="95"/>
-<attribute name="VALUE" x="42.672" y="-20.2438" size="1.778" layer="96"/>
-</instance>
-<instance part="H2" gate="G$1" x="40.64" y="-25.4" smashed="yes">
-<attribute name="NAME" x="42.672" y="-24.8158" size="1.778" layer="95"/>
-<attribute name="VALUE" x="42.672" y="-27.8638" size="1.778" layer="96"/>
-</instance>
-<instance part="H3" gate="G$1" x="40.64" y="-33.02" smashed="yes">
-<attribute name="NAME" x="42.672" y="-32.4358" size="1.778" layer="95"/>
-<attribute name="VALUE" x="42.672" y="-35.4838" size="1.778" layer="96"/>
-</instance>
-<instance part="H4" gate="G$1" x="40.64" y="-40.64" smashed="yes">
-<attribute name="NAME" x="42.672" y="-40.0558" size="1.778" layer="95"/>
-<attribute name="VALUE" x="42.672" y="-43.1038" size="1.778" layer="96"/>
+<instance part="H1" gate="G$1" x="205.74" y="-40.64" smashed="yes">
+<attribute name="NAME" x="207.772" y="-40.0558" size="1.778" layer="95"/>
+<attribute name="VALUE" x="207.772" y="-43.1038" size="1.778" layer="96"/>
+</instance>
+<instance part="H2" gate="G$1" x="205.74" y="-48.26" smashed="yes">
+<attribute name="NAME" x="207.772" y="-47.6758" size="1.778" layer="95"/>
+<attribute name="VALUE" x="207.772" y="-50.7238" size="1.778" layer="96"/>
+</instance>
+<instance part="H3" gate="G$1" x="205.74" y="-55.88" smashed="yes">
+<attribute name="NAME" x="207.772" y="-55.2958" size="1.778" layer="95"/>
+<attribute name="VALUE" x="207.772" y="-58.3438" size="1.778" layer="96"/>
+</instance>
+<instance part="H4" gate="G$1" x="205.74" y="-63.5" smashed="yes">
+<attribute name="NAME" x="207.772" y="-62.9158" size="1.778" layer="95"/>
+<attribute name="VALUE" x="207.772" y="-65.9638" size="1.778" layer="96"/>
+</instance>
+<instance part="P1" gate="G$1" x="45.72" y="-25.4" smashed="yes">
+<attribute name="NAME" x="43.18" y="-22.86" size="1.778" layer="95"/>
+<attribute name="VALUE" x="43.18" y="-31.75" size="1.778" layer="96"/>
+</instance>
+<instance part="P+10" gate="VCC" x="38.1" y="-20.32" smashed="yes">
+<attribute name="VALUE" x="35.56" y="-22.86" size="1.778" layer="96" rot="R90"/>
+</instance>
+<instance part="AGND30" gate="VR1" x="38.1" y="-33.02" smashed="yes">
+<attribute name="VALUE" x="35.56" y="-35.56" size="1.778" layer="96"/>
 </instance>
 </instances>
@@
 <junction x="33.02" y="-76.2"/>
 </segment>
+<segment>
+<pinref part="P1" gate="G$1" pin="2"/>
+<wire x1="40.64" y1="-27.94" x2="38.1" y2="-27.94" width="0.1524" layer="91"/>
+<pinref part="AGND30" gate="VR1" pin="AGND"/>
+<wire x1="38.1" y1="-27.94" x2="38.1" y2="-30.48" width="0.1524" layer="91"/>
+</segment>
 </net>
 <net name="N$2" class="0">
@@
 <wire x1="40.64" y1="-55.88" x2="40.64" y2="-58.42" width="0.1524" layer="91"/>
 </segment>
+<segment>
+<pinref part="P+10" gate="VCC" pin="VCC"/>
+<wire x1="38.1" y1="-22.86" x2="38.1" y2="-25.4" width="0.1524" layer="91"/>
+<pinref part="P1" gate="G$1" pin="1"/>
+<wire x1="38.1" y1="-25.4" x2="40.64" y2="-25.4" width="0.1524" layer="91"/>
+</segment>
 </net>
